File: AlarmUnit/AlarmUnit.sch (KiCad schematic (older format))
At the start: 41 parts, among them J1 Conn_01x12_Male, P1 2K, Q1 BC338, Q2 BC338, Q3 BC338, T1 Transformer_1P_SS, U1 LM324, U2 L7812

Commit message: ya algunos componentes distribuidos en la placa
Parts:
- added C3: 2.2uF, Capacitor_THT:CP_Radial_Tantal_D5.0mm_P2.50mm, symbol Device:CP
- added F1: Fuse, symbol Device:Fuse
- C1, C2: footprint (none) -> Capacitor_THT:CP_Radial_Tantal_D4.5mm_P2.50mm
- C4, C6, C8: footprint (none) -> Capacitor_THT:C_Disc_D5.1mm_W3.2mm_P5.00mm
- C5: footprint (none) -> Capacitor_THT:CP_Axial_L38.0mm_D21.0mm_P44.00mm_Horizontal
- C7: footprint (none) -> Capacitor_THT:CP_Radial_D5.0mm_P2.00mm
- D1: value 6V2 -> 1N825A; footprint (none) -> Diode_THT:D_DO-35_SOD27_P7.62mm_Horizontal
- D2: footprint (none) -> LED_THT:LED_D5.0mm_Horizontal_O6.35mm_Z9.0mm
- D3: footprint (none) -> Diode_THT:D_DO-35_SOD27_P7.62mm_Horizontal
- D4, D5: value D -> 1N4007; footprint (none) -> Diode_THT:D_DO-41_SOD81_P10.16mm_Horizontal
- JP1, JP2, JP3: footprint (none) -> Jumper:SolderJumper-3_P1.3mm_Open_RoundedPad1.0x1.5mm
- P1: footprint (none) -> Potentiometer_THT:Potentiometer_Bourns_3009Y_Horizontal
- R1, R10, R11, R12, R13, R14, R15, R2, R3, R4, R5, R6, R7, R8, R9: footprint (none) -> Resistor_THT:R_Axial_DIN0207_L6.3mm_D2.5mm_P7.62mm_Horizontal
- TP2, TP4: footprint (none) -> TestPoint:TestPoint_Pad_1.0x1.0mm
- U1: footprint (none) -> Package_DIP:DIP-14_W7.62mm
- U2: footprint (none) -> Package_TO_SOT_THT:TO-220-3_Horizontal_TabDown
Connections:
- net +12V: now also C3.2
- net 12: now also F1.2; no longer T1.1 (AA)
- net GND: now also C3.1
- new net: F1.1, T1.1 (AA)
Other:
- note added: "220VAC"
- note added: "IS"
- note added: "SET POINT"
- moved on the sheet: C1, C2, C4, C5, C6, C7, C8, D1, D2, D3, D4, D5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

Commit message: componentes distribuidos a ojo, verificar medidas
Parts:
- added VAC1, VAC2: VAC, TestPoint:TestPoint_Loop_D1.80mm_Drill1.0mm_Beaded, symbol Connector:TestPoint
- added VR1: VR, TestPoint:TestPoint_Loop_D1.80mm_Drill1.0mm_Beaded, symbol Connector:TestPoint
- TP2, TP4: footprint TestPoint:TestPoint_Pad_1.0x1.0mm -> TestPoint:TestPoint_Loop_D1.80mm_Drill1.0mm_Beaded
Connections:
- net VR: now also C5.1, C6.1, D4.1 (K), D5.1 (K), U2.1 (IN), VR1.1
- net at D5.2 (A), T1.3 (SA): now also VAC2.1
- net at D4.2 (A), T1.5 (SB): now also VAC1.1
Changed lines of the file:
@@
 F 0 "TP4" H 6358 3318 50  0000 L CNN
 F 1 "TestPoint" H 6358 3227 50  0000 L CNN
-F 2 "TestPoint:TestPoint_Pad_1.0x1.0mm" H 6500 3200 50  0001 C CNN
+F 2 "TestPoint:TestPoint_Loop_D1.80mm_Drill1.0mm_Beaded" H 6500 3200 50  0001 C CNN
 F 3 "~" H 6500 3200 50  0001 C CNN
 	1    6300 3200
@@
 	-1   0    0    1
 $EndComp
-Text Label 950  6450 0    50   ~ 0
-12
-Text Label 950  6850 0    50   ~ 0
-11
 $Comp
 L power:GND #PWR0115
@@
 F 0 "TP2" H 5458 6768 50  0000 L CNN
 F 1 "TestPoint" H 5458 6677 50  0000 L CNN
-F 2 "TestPoint:TestPoint_Pad_1.0x1.0mm" H 5600 6650 50  0001 C CNN
+F 2 "TestPoint:TestPoint_Loop_D1.80mm_Drill1.0mm_Beaded" H 5600 6650 50  0001 C CNN
 F 3 "~" H 5600 6650 50  0001 C CNN
 	1    5400 6650
@@
 L power:PWR_FLAG #FLG0102
 U 1 1 64DA8C73
-P 3000 6650
-F 0 "#FLG0102" H 3000 6725 50  0001 C CNN
-F 1 "PWR_FLAG" H 3000 6823 50  0000 C CNN
-F 2 "" H 3000 6650 50  0001 C CNN
-F 3 "~" H 3000 6650 50  0001 C CNN
-	1    3000 6650
+P 3300 6650
+F 0 "#FLG0102" H 3300 6725 50  0001 C CNN
+F 1 "PWR_FLAG" H 3300 6823 50  0000 C CNN
+F 2 "" H 3300 6650 50  0001 C CNN
+F 3 "~" H 3300 6650 50  0001 C CNN
+	1    3300 6650
 	1    0    0    -1
 $EndComp
@@
 	3950 3450 3950 3750
 Wire Wire Line
-	3000 6650 3600 6650
+	3000 6650 3300 6650
 Connection ~ 3600 6650
 Wire Wire Line
@@
 $EndComp
 Wire Wire Line
-	1100 6450 950  6450
-Wire Wire Line
-	950  6850 1400 6850
-Wire Wire Line
 	2300 6450 2200 6450
 Wire Wire Line
@@
 Wire Wire Line
 	3350 4250 3350 4400
+Connection ~ 3300 6650
+Wire Wire Line
+	3300 6650 3600 6650
+Wire Wire Line
+	3000 6550 3000 6650
+Text GLabel 3000 6550 1    50   Output ~ 0
+VR
+Connection ~ 2750 6450
+Text Label 950  6850 0    50   ~ 0
+11
+Wire Wire Line
+	950  6850 1400 6850
+Text Label 950  6450 0    50   ~ 0
+12
+Wire Wire Line
+	1100 6450 950  6450
+$Comp
+L Connector:TestPoint VR1
+U 1 1 64F7A7CD
+P 2750 6450
+F 0 "VR1" H 2808 6568 50  0001 L CNN
+F 1 "VR" H 2700 6650 50  0000 L CNN
+F 2 "TestPoint:TestPoint_Loop_D1.80mm_Drill1.0mm_Beaded" H 2950 6450 50  0001 C CNN
+F 3 "~" H 2950 6450 50  0001 C CNN
+	1    2750 6450
+	1    0    0    -1
+$EndComp
+$Comp
+L Connector:TestPoint VAC1
+U 1 1 64F9EC25
+P 2200 6450
+F 0 "VAC1" H 2258 6568 50  0001 L CNN
+F 1 "VAC" H 2150 6650 50  0000 L CNN
+F 2 "TestPoint:TestPoint_Loop_D1.80mm_Drill1.0mm_Beaded" H 2400 6450 50  0001 C CNN
+F 3 "~" H 2400 6450 50  0001 C CNN
+	1    2200 6450
+	1    0    0    -1
+$EndComp
+Connection ~ 2200 6450
+$Comp
+L Connector:TestPoint VAC2
+U 1 1 64FA67ED
+P 2200 6850
+F 0 "VAC2" H 2258 6968 50  0001 L CNN
+F 1 "VAC" H 2150 7050 50  0000 L CNN
+F 2 "TestPoint:TestPoint_Loop_D1.80mm_Drill1.0mm_Beaded" H 2400 6850 50  0001 C CNN
+F 3 "~" H 2400 6850 50  0001 C CNN
+	1    2200 6850
+	-1   0    0    1
+$EndComp
+Connection ~ 2200 6850
 $EndSCHEMATC

Commit message: avances en routeado
Parts:
- RLY1: footprint Relay_THT:Relay_DPDT_Panasonic_JP -> AlarmUnit:Relay_Pana-NC2D-JP-DC24V
Changed lines of the file:
@@
 F 0 "RLY1" V 8817 2200 50  0000 C CNN
 F 1 "NC2D-JP-DC24V" V 8726 2200 50  0000 C CNN
-F 2 "Relay_THT:Relay_DPDT_Panasonic_JP" H 8700 2150 50  0001 L CNN
+F 2 "AlarmUnit:Relay_Pana-NC2D-JP-DC24V" H 8700 2150 50  0000 L CNN
 F 3 "" H 8050 2200 50  0001 C CNN
 	1    8050 2200

Commit message: ruteada placa completa
Parts:
- added GND1: GND, TestPoint:TestPoint_Loop_D1.80mm_Drill1.0mm_Beaded, symbol Connector:TestPoint
- added VAC1, VAC2: VAC, TestPoint:TestPoint_THTPad_D2.5mm_Drill1.2mm, symbol Connector:TestPoint
- J1: footprint (none) -> AlarmUnit:MolexConnBarrierStrip12Pos-953mm
- JP1, JP2, JP3: footprint Jumper:SolderJumper-3_P1.3mm_Open_RoundedPad1.0x1.5mm -> AlarmUnit:WiredJumper
- RLY1: symbol Pana_Relay:NC2D-JP-DC24V -> AlarmUnit-rescue:NC2D-JP-DC24V-Pana_Relay
- renumbered VAC1 to E13, VAC2 to E2
Connections:
- net +12V: now also C3.1; no longer C3.2
- net 11: now also VAC2.1
- net 12: now also VAC1.1
- net GND: now also C3.2, GND1.1; no longer C3.1
- net VR: now also RLY1.4; no longer RLY1.5
- net at D3.2 (A), Q2.1 (C): now also RLY1.5; no longer RLY1.4
Changed lines of the file:
@@
 F 0 "J1" V 8385 628 50  0000 C CNN
 F 1 "Conn_01x12_Male" V 8476 628 50  0000 C CNN
-F 2 "" H 8550 700 50  0001 C CNN
+F 2 "AlarmUnit:MolexConnBarrierStrip12Pos-953mm" H 8550 700 50  0001 C CNN
 F 3 "~" H 8550 700 50  0001 C CNN
 	1    8550 700
@@
 	4500 4800 4300 4800
 $Comp
-L Pana_Relay:NC2D-JP-DC24V RLY1
+L AlarmUnit-rescue:NC2D-JP-DC24V-Pana_Relay RLY1
 U 1 1 64E6AA08
 P 8050 2200
@@
 F 0 "JP1" V 7246 1812 50  0000 R CNN
 F 1 "Jumper" V 7155 1812 50  0000 R CNN
-F 2 "Jumper:SolderJumper-3_P1.3mm_Open_RoundedPad1.0x1.5mm" H 7200 1900 50  0001 C CNN
+F 2 "AlarmUnit:WiredJumper" H 7200 1900 50  0001 C CNN
 F 3 "~" H 7200 1900 50  0001 C CNN
 	1    7200 1900
@@
 F 0 "JP2" V 9196 1712 50  0000 R CNN
 F 1 "Jumper" V 9105 1712 50  0000 R CNN
-F 2 "Jumper:SolderJumper-3_P1.3mm_Open_RoundedPad1.0x1.5mm" H 9150 1800 50  0001 C CNN
+F 2 "AlarmUnit:WiredJumper" H 9150 1800 50  0001 C CNN
 F 3 "~" H 9150 1800 50  0001 C CNN
 	1    9150 1800
@@
 F 0 "JP3" V 9496 1912 50  0000 R CNN
 F 1 "Jumper" V 9405 1912 50  0000 R CNN
-F 2 "Jumper:SolderJumper-3_P1.3mm_Open_RoundedPad1.0x1.5mm" H 9450 2000 50  0001 C CNN
+F 2 "AlarmUnit:WiredJumper" H 9450 2000 50  0001 C CNN
 F 3 "~" H 9450 2000 50  0001 C CNN
 	1    9450 2000
@@
 Connection ~ 4250 6950
 Wire Wire Line
-	4250 6950 4900 6950
+	4250 6950 4600 6950
 $Comp
 L power:GND #PWR0106
@@
 Wire Wire Line
 	4250 6950 4250 7000
-Wire Wire Line
-	3350 4050 3350 4250
 Wire Wire Line
 	3950 6650 3600 6650
@@
 Text Notes 750  6650 0    50   ~ 0
 220VAC
+Wire Wire Line
+	2300 6450 2200 6450
+Wire Wire Line
+	2300 6850 2200 6850
+$Comp
+L Device:CP C3
+U 1 1 64E90DCF
+P 3500 4250
+F 0 "C3" V 3245 4250 50  0000 C CNN
+F 1 "2.2uF" V 3336 4250 50  0000 C CNN
+F 2 "Capacitor_THT:CP_Radial_Tantal_D5.0mm_P2.50mm" H 3538 4100 50  0001 C CNN
+F 3 "~" H 3500 4250 50  0001 C CNN
+	1    3500 4250
+	0    -1   -1   0
+$EndComp
+$Comp
+L power:GND #PWR0113
+U 1 1 64E91F7B
+P 3650 4250
+F 0 "#PWR0113" H 3650 4000 50  0001 C CNN
+F 1 "GND" H 3655 4077 50  0000 C CNN
+F 2 "" H 3650 4250 50  0001 C CNN
+F 3 "" H 3650 4250 50  0001 C CNN
+	1    3650 4250
+	1    0    0    -1
+$EndComp
+Connection ~ 3350 4250
+Connection ~ 3300 6650
+Wire Wire Line
+	3300 6650 3600 6650
+Wire Wire Line
+	3000 6550 3000 6650
+Text GLabel 3000 6550 1    50   Output ~ 0
+VR
+Connection ~ 2750 6450
+Text Label 950  6850 0    50   ~ 0
+11
+Wire Wire Line
+	950  6850 1400 6850
+Text Label 950  6450 0    50   ~ 0
+12
+Wire Wire Line
+	1100 6450 950  6450
+$Comp
+L Connector:TestPoint VR1
+U 1 1 64F7A7CD
+P 2750 6450
+F 0 "VR1" H 2808 6568 50  0001 L CNN
+F 1 "VR" H 2700 6650 50  0000 L CNN
+F 2 "TestPoint:TestPoint_Loop_D1.80mm_Drill1.0mm_Beaded" H 2950 6450 50  0001 C CNN
+F 3 "~" H 2950 6450 50  0001 C CNN
+	1    2750 6450
+	1    0    0    -1
+$EndComp
+$Comp
+L Connector:TestPoint E13
+U 1 1 64F9EC25
+P 2200 6450
+F 0 "E13" H 2258 6568 50  0001 L CNN
+F 1 "VAC" H 2150 6650 50  0000 L CNN
+F 2 "TestPoint:TestPoint_Loop_D1.80mm_Drill1.0mm_Beaded" H 2400 6450 50  0001 C CNN
+F 3 "~" H 2400 6450 50  0001 C CNN
+	1    2200 6450
+	1    0    0    -1
+$EndComp
+Connection ~ 2200 6450
+$Comp
+L Connector:TestPoint E2
+U 1 1 64FA67ED
+P 2200 6850
+F 0 "E2" H 2258 6968 50  0001 L CNN
+F 1 "VAC" H 2150 7050 50  0000 L CNN
+F 2 "TestPoint:TestPoint_Loop_D1.80mm_Drill1.0mm_Beaded" H 2400 6850 50  0001 C CNN
+F 3 "~" H 2400 6850 50  0001 C CNN
+	1    2200 6850
+	-1   0    0    1
+$EndComp
+Connection ~ 2200 6850
+Wire Wire Line
+	3350 4050 3350 4250
+Wire Wire Line
+	3350 4250 3350 4400
+$Comp
+L Connector:TestPoint GND1
+U 1 1 64E15C9F
+P 4600 6950
+F 0 "GND1" H 4658 7068 50  0001 L CNN
+F 1 "GND" H 4550 7150 50  0000 L CNN
+F 2 "TestPoint:TestPoint_Loop_D1.80mm_Drill1.0mm_Beaded" H 4800 6950 50  0001 C CNN
+F 3 "~" H 4800 6950 50  0001 C CNN
+	1    4600 6950
+	1    0    0    -1
+$EndComp
+Connection ~ 4600 6950
+Wire Wire Line
+	4600 6950 4900 6950
+$Comp
+L Connector:TestPoint VAC1
+U 1 1 64E240EF
+P 950 6450
+F 0 "VAC1" H 1008 6568 50  0001 L CNN
+F 1 "VAC" H 900 6650 50  0000 L CNN
+F 2 "TestPoint:TestPoint_THTPad_D2.5mm_Drill1.2mm" H 1150 6450 50  0001 C CNN
+F 3 "~" H 1150 6450 50  0001 C CNN
+	1    950  6450
+	0    -1   -1   0
+$EndComp
 $Comp
 L Device:Fuse F1
@@
 	0    1    1    0
 $EndComp
-Wire Wire Line
-	2300 6450 2200 6450
-Wire Wire Line
-	2300 6850 2200 6850
-$Comp
-L Device:CP C3
-U 1 1 64E90DCF
-P 3500 4250
-F 0 "C3" V 3245 4250 50  0000 C CNN
-F 1 "2.2uF" V 3336 4250 50  0000 C CNN
-F 2 "Capacitor_THT:CP_Radial_Tantal_D5.0mm_P2.50mm" H 3538 4100 50  0001 C CNN
-F 3 "~" H 3500 4250 50  0001 C CNN
-	1    3500 4250
-	0    1    1    0
-$EndComp
-$Comp
-L power:GND #PWR0113
-U 1 1 64E91F7B
-P 3650 4250
-F 0 "#PWR0113" H 3650 4000 50  0001 C CNN
-F 1 "GND" H 3655 4077 50  0000 C CNN
-F 2 "" H 3650 4250 50  0001 C CNN
-F 3 "" H 3650 4250 50  0001 C CNN
-	1    3650 4250
-	1    0    0    -1
-$EndComp
-Connection ~ 3350 4250
-Wire Wire Line
-	3350 4250 3350 4350
-Wire Wire Line
-	3350 4250 3350 4400
-Connection ~ 3300 6650
-Wire Wire Line
-	3300 6650 3600 6650
-Wire Wire Line
-	3000 6550 3000 6650
-Text GLabel 3000 6550 1    50   Output ~ 0
-VR
-Connection ~ 2750 6450
-Text Label 950  6850 0    50   ~ 0
-11
-Wire Wire Line
-	950  6850 1400 6850
-Text Label 950  6450 0    50   ~ 0
-12
-Wire Wire Line
-	1100 6450 950  6450
-$Comp
-L Connector:TestPoint VR1
-U 1 1 64F7A7CD
-P 2750 6450
-F 0 "VR1" H 2808 6568 50  0001 L CNN
-F 1 "VR" H 2700 6650 50  0000 L CNN
-F 2 "TestPoint:TestPoint_Loop_D1.80mm_Drill1.0mm_Beaded" H 2950 6450 50  0001 C CNN
-F 3 "~" H 2950 6450 50  0001 C CNN
-	1    2750 6450
-	1    0    0    -1
-$EndComp
-$Comp
-L Connector:TestPoint VAC1
-U 1 1 64F9EC25
-P 2200 6450
-F 0 "VAC1" H 2258 6568 50  0001 L CNN
-F 1 "VAC" H 2150 6650 50  0000 L CNN
-F 2 "TestPoint:TestPoint_Loop_D1.80mm_Drill1.0mm_Beaded" H 2400 6450 50  0001 C CNN
-F 3 "~" H 2400 6450 50  0001 C CNN
-	1    2200 6450
-	1    0    0    -1
-$EndComp
-Connection ~ 2200 6450
 $Comp
 L Connector:TestPoint VAC2
-U 1 1 64FA67ED
-P 2200 6850
-F 0 "VAC2" H 2258 6968 50  0001 L CNN
-F 1 "VAC" H 2150 7050 50  0000 L CNN
-F 2 "TestPoint:TestPoint_Loop_D1.80mm_Drill1.0mm_Beaded" H 2400 6850 50  0001 C CNN
-F 3 "~" H 2400 6850 50  0001 C CNN
-	1    2200 6850
-	-1   0    0    1
-$EndComp
-Connection ~ 2200 6850
+U 1 1 64E348EE
+P 950 6850
+F 0 "VAC2" H 1008 6968 50  0001 L CNN
+F 1 "VAC" H 900 7050 50  0000 L CNN
+F 2 "TestPoint:TestPoint_THTPad_D2.5mm_Drill1.2mm" H 1150 6850 50  0001 C CNN
+F 3 "~" H 1150 6850 50  0001 C CNN
+	1    950  6850
+	0    -1   -1   0
+$EndComp
 $EndSCHEMATC
