File: AlarmUnit/AlarmUnit.kicad_pcb (KiCad board)
At the start: 2 copper layers, 39 parts, among them P1 2K, Q1 BC338, Q2 BC338, Q3 BC338, U1 LM324, U2 L7812

Commit message: componentes distribuidos a ojo, verificar medidas
Parts:
- added VAC1: VAC, TestPoint:TestPoint_Loop_D1.80mm_Drill1.0mm_Beaded, F.Cu at (240.0, 115.6)
- added VAC2: VAC, TestPoint:TestPoint_Loop_D1.80mm_Drill1.0mm_Beaded, F.Cu at (232.4, 129.5)
- added VR1: VR, TestPoint:TestPoint_Loop_D1.80mm_Drill1.0mm_Beaded, F.Cu at (194.3, 110.5)
- TP2, TP4: footprint TestPoint:TestPoint_Pad_1.0x1.0mm -> TestPoint:TestPoint_Loop_D1.80mm_Drill1.0mm_Beaded
- moved D5 6.35 mm to (222.2, 121.9)
- moved D4 5.08 mm to (222.2, 115.6)
Connections:
- C5 pad 1: Net-(C5-Pad1) -> VR
- C6 pad 1: Net-(C5-Pad1) -> VR
- D4 pad 1: Net-(C5-Pad1) -> VR
- D5 pad 1: Net-(C5-Pad1) -> VR
- U2 pad 1: Net-(C5-Pad1) -> VR
Routing:
- net (no net): vias 0 -> 4
Other:
- board outline added: 184.2 x 102.9 mm

Commit message: avances en routeado
Parts:
- added RLY1: NC2D-JP-DC24V, AlarmUnit:Relay_Pana-NC2D-JP-DC24V, F.Cu at (174.0, 76.2)
- moved JP1 16.7 mm to (203.2, 59.7)
- moved JP2 16.7 mm to (203.2, 49.5)
- moved JP3 16.7 mm to (203.2, 54.6)
- moved R12 12.6 mm to (156.2, 95.2)
- moved R11 11.7 mm to (151.1, 95.2)
- moved Q3 11.7 mm to (128.3, 96.5)
- moved R8 9.16 mm to (119.4, 90.2)
- moved TP2 9.16 mm to (115.6, 104.1)
- moved R15 9.16 mm to (111.8, 96.5)
- moved C1 7.62 mm to (147.3, 44.5)
- moved C2 7.62 mm to (119.4, 78.7)
- moved C3 7.62 mm to (153.7, 67.3)
- moved C4 7.62 mm to (138.4, 44.5)
- moved Q1 7.62 mm to (165.1, 88.9)
- moved R1 7.62 mm to (138.4, 52.1)
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Routing:
- net +12V: track 0.00 -> 165.0 mm
- net VR: track 0.00 -> 126.0 mm
- net Net-(JP3-Pad1): track 0.00 -> 45.8 mm
- net Net-(R8-Pad1): track 0.00 -> 43.3 mm
- net Net-(JP2-Pad1): track 0.00 -> 37.1 mm
- net Net-(R10-Pad1): track 0.00 -> 36.1 mm
- net GND: track 0.00 -> 20.2 mm
- net Net-(D1-Pad1): track 0.00 -> 15.2 mm
- net Net-(R7-Pad2): track 0.00 -> 11.4 mm
- net Net-(D5-Pad2): track 0.00 -> 8.89 mm
- net Net-(D4-Pad2): track 0.00 -> 7.62 mm
- net Net-(D3-Pad2): track 0.00 -> 6.35 mm
Other:
- net class Double added: clearance 0.2, trace_width 0.5, via_dia 0.8, via_drill 0.4

Commit message: ruteada placa completa
Parts:
- added GND1: GND, TestPoint:TestPoint_Loop_D1.80mm_Drill1.0mm_Beaded, F.Cu at (222.2, 125.7)
- added J1: Conn_01x12_Male, AlarmUnit:MolexConnBarrierStrip12Pos-953mm, F.Cu at (126.3, 36.8)
- added VAC1: VAC, TestPoint:TestPoint_THTPad_D2.5mm_Drill1.2mm, F.Cu at (231.1, 43.2)
- added VAC2: VAC, TestPoint:TestPoint_THTPad_D2.5mm_Drill1.2mm, F.Cu at (221.6, 43.2)
- JP1, JP2, JP3: footprint Jumper:SolderJumper-3_P1.3mm_Open_RoundedPad1.0x1.5mm -> AlarmUnit:WiredJumper
- moved D1 14.0 mm to (73.7, 39.4)
- moved R1 8.98 mm to (147.3, 50.8), turned to 180 degrees
- moved P1 8.89 mm to (81.3, 49.5)
- moved R5 8.89 mm to (81.3, 59.7)
- moved R6 8.89 mm to (73.7, 54.6)
- moved JP3 3.81 mm to (199.4, 54.6)
- moved R13 3.81 mm to (174.0, 94.0)
- moved JP1 3.81 mm to (199.4, 59.7)
- moved JP2 3.81 mm to (199.4, 49.5)
- moved R4 3.59 mm to (129.5, 64.8)
- moved R8 2.84 mm to (120.7, 87.6)
- moved R15 2.84 mm to (113.0, 94.0)
- moved Q3 2.84 mm to (129.5, 94.0), turned to 270 degrees
- moved C2 2.54 mm to (121.9, 78.7)
- moved Q1 2.54 mm to (165.1, 86.4), turned to 270 degrees
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- renumbered VAC1 to E13, VAC2 to E2
Connections:
- C3 pad 1: GND -> +12V
- C3 pad 2: +12V -> GND
Routing:
- net GND: track 20.2 -> 410.4 mm
- net VR: track 126.0 -> 390.4 mm
- net +12V: track 165.0 -> 290.3 mm
- net Net-(P1-Pad2): track 0.00 -> 104.3 mm
- net Net-(D2-Pad1): track 0.00 -> 71.4 mm
- net /7: track 0.00 -> 57.8 mm
- net /2: track 0.00 -> 43.1 mm
- net Net-(JP1-Pad1): track 0.00 -> 42.2 mm
- net Net-(C4-Pad1): track 0.00 -> 34.1 mm
- net /5: track 0.00 -> 29.3 mm
- net /10: track 0.00 -> 29.2 mm
- net /8: track 0.00 -> 26.0 mm
- net Net-(C2-Pad1): track 0.00 -> 25.9 mm
- net Net-(R4-Pad1): track 0.00 -> 25.2 mm
- net Net-(C1-Pad1): track 0.00 -> 19.4 mm
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Other:
- board size 184.2 x 102.9 mm -> 184.2 x 106.7 mm

Commit message: algunos tweaks
Parts:
- moved Q3 1.91 mm to (129.5, 95.9)
- moved R11 1.91 mm to (152.4, 97.2)
- moved R12 1.91 mm to (157.5, 97.2)
- moved R15 1.91 mm to (113.0, 95.9)
Routing:
- net Net-(R10-Pad1): track 36.1 -> 45.0 mm
- net Net-(P1-Pad2): track 104.3 -> 107.9 mm
- net Net-(D3-Pad2): track 25.0 -> 28.2 mm
- net /7: track 57.8 -> 60.1 mm
- net Net-(D2-Pad1): track 71.4 -> 73.7 mm
- net GND: track 410.4 -> 408.5 mm
- net +12V: track 290.3 -> 288.4 mm
- net VR: track 390.4 -> 389.7 mm
- net (no net): vias 4 -> 6
